File: BTM308-host/BTM308-host.kicad_pcb (KiCad board)
At the start: 2 copper layers, 41 parts, among them J1 Audio OUT, J2 USB_C_Receptacle_USB2.0_16P, J3 Battery Connector, U1 Bluetooth Module, U2 OPA1678

Commit message: layout position set
Parts:
- added J4: Battery -, Connector_PinHeader_2.54mm:PinHeader_1x01_P2.54mm_Vertical, F.Cu at (165.3, 93.8)
- added J5: Top, Connector_PinHeader_2.54mm:PinHeader_2x04_P2.54mm_Vertical, F.Cu at (127.9, 85.0)
- added J6: Battery +, Connector_PinHeader_2.54mm:PinHeader_1x01_P2.54mm_Vertical, F.Cu at (117.5, 83.5)
- added J7: Battery -, Connector_PinHeader_2.54mm:PinHeader_1x01_P2.54mm_Vertical, F.Cu at (117.5, 79.3)
- added SW1: PLAY, TS-A002:TST-A002_0.6MM_BOSS, F.Cu at (117.0, 58.8)
- added SW2: VOL+, TS-A002:TST-A002_0.6MM_BOSS, F.Cu at (116.9, 65.0)
- added SW3: VOL-, TS-A002:TST-A002_0.6MM_BOSS, F.Cu at (117.0, 71.3)
- added SW4: ON/OFF, KiCad:SLW8645745ARAND, F.Cu at (129.1, 93.0)
- added SW6: Battery Status, TS-A002:TST-A002_0.6MM_BOSS, F.Cu at (117.1, 92.5)
- added U3: PJ-320A, PJ-320A_Library:PJ-320A, F.Cu at (169.2, 62.2)
- J1: value Audio OUT -> Bottom; footprint Connector_PinHeader_2.54mm:PinHeader_1x03_P2.54mm_Vertical -> Connector_PinSocket_2.54mm:PinSocket_2x04_P2.54mm_Vertical
- J3: value Battery Connector -> Battery +; footprint Connector_JST:JST_XH_S2B-XH-A_1x02_P2.50mm_Horizontal -> Connector_PinHeader_2.54mm:PinHeader_1x01_P2.54mm_Vertical
- moved D2 73.8 mm to (121.6, 86.8), turned to -90 degrees
- moved D1 70.9 mm to (124.1, 86.8), turned to -90 degrees
- moved C9 35.0 mm to (166.0, 78.2), turned to 90 degrees
- moved C10 34.0 mm to (163.8, 78.2), turned to -90 degrees
- moved C1 31.9 mm to (162.2, 91.0), turned to -90 degrees
- moved D3 31.8 mm to (158.0, 91.7), turned to -90 degrees
- moved R17 31.4 mm to (145.8, 85.7), turned to 90 degrees
- moved R11 29.4 mm to (166.0, 74.2), turned to 90 degrees
- moved R13 28.6 mm to (163.8, 74.2), turned to -90 degrees
- moved J1 28.5 mm to (157.7, 82.6), turned to 90 degrees
- moved R4 28.1 mm to (121.6, 82.3), turned to -90 degrees
- moved R18 28.0 mm to (148.0, 85.7), turned to 90 degrees
- moved R16 25.6 mm to (152.8, 78.2), turned to 90 degrees
- moved R5 24.2 mm to (124.1, 82.3), turned to -90 degrees
- moved R3 23.8 mm to (120.4, 71.3), turned to 90 degrees
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Connections:
- C11 pad 2: Net-(J1-Pin_2) -> Net-(U3-Ring1)
- C2 pad 2: Net-(J1-Pin_1) -> Net-(U3-Tip)
- J1 pad 1: Net-(J1-Pin_1) -> GND
- J1 pad 2: Net-(J1-Pin_2) -> /VBAT
- J1 pad 3: AGND -> /VCHG
- R19 pad 2: Net-(J1-Pin_2) -> Net-(U3-Ring1)
- R20 pad 2: Net-(J1-Pin_1) -> Net-(U3-Tip)
- U1 pad 39: GND -> AGND
Other:
- board outline added: 52.8 x 40.1 mm
- copper layers 2 -> 4
