File: BTM308-host/BTM308-host.kicad_sch (KiCad schematic)
At the start: 45 parts, among them J1 Audio OUT, J2 USB_C_Receptacle_USB2.0_16P, SW1 PLAY, SW2 VOL+, SW3 VOL-, SW4 ON/OFF, U2 OPA1678

Commit message: schematic finished
Parts:
- removed JP1: SPI/PCM, symbol Jumper:Jumper_3_Open
- added J3: Battery Connector, Connector_JST:JST_XH_S2B-XH-A_1x02_P2.50mm_Horizontal, symbol Connector:Conn_01x02_Socket
- C1, C10, C11, C12, C13, C2, C3, C4, C5, C6, C7, C8, C9: footprint (none) -> Capacitor_SMD:C_0805_2012Metric_Pad1.18x1.45mm_HandSolder
- D1, D2: footprint (none) -> LED_SMD:LED_0805_2012Metric_Pad1.15x1.40mm_HandSolder
- J1: footprint (none) -> Connector_PinHeader_2.54mm:PinHeader_1x03_P2.54mm_Vertical
- J2: footprint (none) -> Connector_USB:USB_C_Receptacle_HRO_TYPE-C-31-M-12
- R1, R10, R11, R12, R13, R14, R15, R16, R17, R18, R19, R2, R20, R3, R4, R5, R6, R7, R8, R9: footprint (none) -> Resistor_SMD:R_0805_2012Metric_Pad1.20x1.40mm_HandSolder
- U1: value ~ -> Bluetooth Module; footprint (none) -> BTM308:BTM308
- U2: footprint (none) -> Package_SO:SOIC-8_5.3x5.3mm_P1.27mm
Connections:
- net GND: now also U1.16 (GND), U1.25 (GND), U1.39 (GND), J3.2 (Pin_2); no longer U1. (VCHG)
- net LED0: now also U1.27 (LED0); no longer U1. (VCHG)
- net LED2: now also U1.28 (LED2); no longer U1. (VCHG)
- net MFB: now also U1.29 (MFB); no longer U1. (VCHG)
- net SPK_AN: now also U1.37 (SPK_AN); no longer U1. (VCHG)
- net SPK_AP: now also U1.38 (SPK_AP); no longer U1. (VCHG)
- net SPK_BN: now also U1.35 (SPK_BN)
- net SPK_BP: now also U1.36 (SPK_BP); no longer U1. (VCHG)
- net VBAT: now also U1.26 (VBAT), J3.1 (Pin_1); no longer U1. (VCHG)
- net VCHG: now also U1.24 (VCHG); no longer U1. (VCHG)
- net at SW1.1, SW2.1, SW3.1: now also U1.9 (1V8); no longer U1. (VCHG)
- net at R3.2: now also U1.3 (PIO0); no longer U1. (VCHG)
- net at R1.2: now also U1.1 (PIO8); no longer U1. (VCHG)
- net at R2.2: now also U1.2 (PIO1); no longer U1. (VCHG)
- no-connect marks 23 -> 28
Other:
- moved on the sheet: D1, D2, R4, R5, SW4

Commit message: layout position set
Parts:
- removed J1: Audio OUT, Connector_PinHeader_2.54mm:PinHeader_1x03_P2.54mm_Vertical, symbol Connector:Conn_01x03_Socket
- removed J3: Battery Connector, Connector_JST:JST_XH_S2B-XH-A_1x02_P2.50mm_Horizontal, symbol Connector:Conn_01x02_Socket
- added J1: Bottom, Connector_PinSocket_2.54mm:PinSocket_2x04_P2.54mm_Vertical, symbol Connector_Generic:Conn_02x04_Top_Bottom
- added J3, J6: Battery +, Connector_PinHeader_2.54mm:PinHeader_1x01_P2.54mm_Vertical, symbol Connector:Conn_01x01_Socket
- added J4, J7: Battery -, Connector_PinHeader_2.54mm:PinHeader_1x01_P2.54mm_Vertical, symbol Connector:Conn_01x01_Socket
- added J5: Top, Connector_PinHeader_2.54mm:PinHeader_2x04_P2.54mm_Vertical, symbol Connector_Generic:Conn_02x04_Top_Bottom
- added SW6: Battery Status, TS-A002:TST-A002_0.6MM_BOSS, symbol Switch:SW_Push
- added U3: PJ-320A, PJ-320A_Library:PJ-320A, symbol PJ-320A_Library:PJ-320A
- SW1, SW2, SW3: footprint (none) -> TS-A002:TST-A002_0.6MM_BOSS
- SW4: footprint (none) -> KiCad:SLW8645745ARAND
Connections:
- net AGND: now also U1.39 (GND), J1.4 (Pin_4), J5.4 (Pin_4), U3.1 (Sleeve)
- net GND: now also J1.1 (Pin_1), J4.1 (Pin_1), J5.1 (Pin_1), J7.1 (Pin_1); no longer U1.39 (GND)
- net SPK_AN: now also J1.6 (Pin_6), J5.6 (Pin_6)
- net SPK_AP: now also J1.5 (Pin_5), J5.5 (Pin_5)
- net SPK_BN: now also J1.8 (Pin_8), J5.8 (Pin_8)
- net SPK_BP: now also J1.7 (Pin_7), J5.7 (Pin_7)
- net VBAT: now also J1.2 (Pin_2), J3.1 (Pin_1), J5.2 (Pin_2), SW6.1
- net VCHG: now also J1.3 (Pin_3), J5.3 (Pin_3)
- net at C11.2, R19.2: now also U3.3 (Ring1)
- net at C2.2, R20.2: now also U3.2 (Tip)
- new net: J6.1 (Pin_1), SW6.2
- no-connect marks 28 -> 29
Other:
- note added: "Battery Status Connection"
- note added: "Board to Board Connection"
- note added: "T: Left R: Right S: GND"
- moved on the sheet: C1, D1, D2, D3, J2, R1, R17, R18, R2, R3, R4, R5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

Commit message: layout done
Parts:
- added R21: 0, Resistor_SMD:R_0805_2012Metric_Pad1.20x1.40mm_HandSolder, symbol Device:R
- J1: footprint Connector_PinSocket_2.54mm:PinSocket_2x04_P2.54mm_Vertical -> Connector_PinHeader_2.54mm:PinHeader_2x05_P2.54mm_Vertical; symbol Connector_Generic:Conn_02x04_Top_Bottom -> Connector_Generic:Conn_02x05_Odd_Even
- J5: footprint Connector_PinHeader_2.54mm:PinHeader_2x04_P2.54mm_Vertical -> Connector_PinHeader_2.54mm:PinHeader_2x05_P2.54mm_Vertical; symbol Connector_Generic:Conn_02x04_Top_Bottom -> Connector_Generic:Conn_02x05_Odd_Even
- SW2: value VOL+ -> VOL-
- SW3: value VOL- -> VOL+
Connections:
- net AGND: now also J1.1 (Pin_1), J1.2 (Pin_2), J1.3 (Pin_3), J5.1 (Pin_1), J5.2 (Pin_2), J5.3 (Pin_3); no longer J1.4 (Pin_4), J5.4 (Pin_4), U3.1 (Sleeve)
- net GND: now also J1.5 (Pin_5), J5.5 (Pin_5), U3.1 (Sleeve); no longer J1.1 (Pin_1), J5.1 (Pin_1)
- net SPK_AN: now also J1.4 (Pin_4), J5.4 (Pin_4); no longer J1.6 (Pin_6), J5.6 (Pin_6)
- net SPK_AP: now also J1.6 (Pin_6), J5.6 (Pin_6); no longer J1.5 (Pin_5), J5.5 (Pin_5)
- net SPK_BN: now also J1.10 (Pin_10), J5.10 (Pin_10); no longer J1.8 (Pin_8), J5.8 (Pin_8)
- net SPK_BP: now also J1.8 (Pin_8), J5.8 (Pin_8); no longer J1.7 (Pin_7), J5.7 (Pin_7)
- net VBAT: now also J1.9 (Pin_9), J5.9 (Pin_9), R21.1; no longer J1.2 (Pin_2), J5.2 (Pin_2), U2.8 (V+)
- net VCHG: now also J1.7 (Pin_7), J5.7 (Pin_7); no longer J1.3 (Pin_3), J5.3 (Pin_3)
- net 1V8: now reaches SW1.1, SW2.1, SW3.1, U1.9 (1V8)
- new net: R21.2, U2.8 (V+)
Other:
- note added: "Ferrite Bead"
- moved on the sheet: C3, C4, U2C
