File: BTM308-host/BTM308-host-bottom/BTM308-host-bottom.kicad_pcb (KiCad board)
At the start: 4 copper layers, 52.8 x 40.1 mm, 52 parts, among them J1 Bottom, J2 USB_C_Receptacle_USB2.0_16P, J3 Battery +, J4 Battery -, J5 Top, J6 Battery +, J7 Battery -, SW1 PLAY, SW2 VOL-, SW3 VOL+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

Commit message: fab
Parts:
- removed D1: BLUE, LED_SMD:LED_0805_2012Metric_Pad1.15x1.40mm_HandSolder
- removed D2: RED, LED_SMD:LED_0805_2012Metric_Pad1.15x1.40mm_HandSolder
- removed J5: Top, Connector_PinHeader_2.54mm:PinHeader_2x05_P2.54mm_Vertical
- removed J6: Battery +, Connector_PinHeader_2.54mm:PinHeader_1x01_P2.54mm_Vertical
- removed J7: Battery -, Connector_PinHeader_2.54mm:PinHeader_1x01_P2.54mm_Vertical
- removed R1, R2, R3, R4, R5: 1k, Resistor_SMD:R_0805_2012Metric_Pad1.20x1.40mm_HandSolder
- removed SW1: PLAY, TS-A002:TST-A002_0.6MM_BOSS
- removed SW2: VOL-, TS-A002:TST-A002_0.6MM_BOSS
- removed SW3: VOL+, TS-A002:TST-A002_0.6MM_BOSS
- removed SW4: ON/OFF, KiCad:SLW8645745ARAND
- removed SW6: Battery Status, TS-A002:TST-A002_0.6MM_BOSS
- removed U1: Bluetooth Module, BTM308:BTM308
Routing:
- net AGND: track 54.3 -> 14.4 mm, vias 14 -> 10
- net /MFB: track 36.4 -> 0.00 mm, vias 1 -> 0
- net /SPK_AP: track 37.6 -> 7.99 mm, vias 1 -> 0
- net /SPK_AN: track 36.5 -> 7.12 mm, vias 1 -> 0
- net /LED2: track 29.0 -> 0.00 mm, vias 2 -> 0
- net /1V8: track 28.3 -> 0.00 mm
- net /LED0: track 28.0 -> 0.00 mm, vias 2 -> 0
- net /SPK_BP: track 31.4 -> 7.10 mm, vias 1 -> 0
- net /SPK_BN: track 32.2 -> 7.97 mm, vias 1 -> 0
- net Net-(U1-PIO1): track 17.0 -> 0.00 mm, vias 2 -> 0
- net /VCHG: track 20.6 -> 6.18 mm
- net Net-(U1-PIO8): track 12.4 -> 0.00 mm, vias 2 -> 0
- net Net-(U1-PIO0): track 9.89 -> 0.00 mm, vias 2 -> 0
- net /VBAT: track 39.3 -> 32.4 mm, vias 6 -> 1
- net Net-(J6-Pin_1): track 5.48 -> 0.00 mm
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Other:
- board size 52.8 x 40.1 mm -> 23 x 40 mm
- board text added: "JLCJLCJLCJLC"
- board text removed: "Battery Status"
